Commit message: added a reference point in the robot urdf

File: hexapod_pkg/urdf/hexapod_still.urdf (robot description, URDF)
Before this commit: robot hexapod, 25 links, 24 joints
Links:
- removed link foot_link_1_tipple
- removed link foot_link_2_tipple
- removed link foot_link_3_tipple
- removed link foot_link_4_tipple
- removed link foot_link_5_tipple
- removed link foot_link_6_tipple
Joints:
- removed joint joint_1_tipple
- removed joint joint_2_tipple
- removed joint joint_3_tipple
- removed joint joint_4_tipple
- removed joint joint_5_tipple
- removed joint joint_6_tipple
- added joint world_joint: type fixed, parent world, child base_link, origin xyz=0 0 0 rpy=0 0 0
