Commit message: changed the self.max_angular_v, kp, kd in HexapodRobotPose

File: hexapod_pkg/urdf/hexapod.urdf (robot description, URDF)
Before this commit: robot hexapod, 25 links, 24 joints
Links:
- removed link foot_link_1_tipple
- removed link foot_link_2_tipple
- removed link foot_link_3_tipple
- removed link foot_link_4_tipple
- removed link foot_link_5_tipple
- removed link foot_link_6_tipple
- added link foot_link_1t; visual sphere radius=0.0001
- added link foot_link_2t; visual sphere radius=0.0001
- added link foot_link_3t; visual sphere radius=0.0001
- added link foot_link_4t; visual sphere radius=0.0001
- added link foot_link_5t; visual sphere radius=0.0001
- added link foot_link_6t; visual sphere radius=0.0001
Joints:
- removed joint joint_1_tipple
- removed joint joint_2_tipple
- removed joint joint_3_tipple
- removed joint joint_4_tipple
- removed joint joint_5_tipple
- removed joint joint_6_tipple
- added joint joint_1t: type revolute, parent foot_link_13, child foot_link_1t, origin xyz=0 0.15209 -0.04637 rpy=0 0 0, axis 0 0 1, limit lower=-0.001 upper=0.001 effort=0.1 velocity=3.0
- added joint joint_2t: type revolute, parent foot_link_23, child foot_link_2t, origin xyz=-0.15209 0 -0.04637 rpy=0 0 0, axis 0 0 1, limit lower=-0.001 upper=0.001 effort=0.1 velocity=3.0
- added joint joint_3t: type revolute, parent foot_link_33, child foot_link_3t, origin xyz=0 -0.15209 -0.04637 rpy=0 0 0, axis 0 0 1, limit lower=-0.001 upper=0.001 effort=0.1 velocity=3.0
- added joint joint_4t: type revolute, parent foot_link_43, child foot_link_4t, origin xyz=0 0.15209 -0.04637 rpy=0 0 0, axis 0 0 1, limit lower=-0.001 upper=0.001 effort=0.1 velocity=3.0
- added joint joint_5t: type revolute, parent foot_link_53, child foot_link_5t, origin xyz=0.15209 0 -0.04637 rpy=0 0 0, axis 0 0 1, limit lower=-0.001 upper=0.001 effort=0.1 velocity=3.0
- added joint joint_6t: type revolute, parent foot_link_63, child foot_link_6t, origin xyz=0 -0.15209 -0.04637 rpy=0 0 0, axis 0 0 1, limit lower=-0.001 upper=0.001 effort=0.1 velocity=3.0
